File: pcb/pcb_f730/pcb_f730.sch (KiCad schematic (older format))
At the start: 67 parts

Commit message: update schematics
Parts:
- removed J?: Micro_SD_Card_Det, symbol Connector:Micro_SD_Card_Det
- removed J? (x2): Conn_01x13, symbol Connector_Generic:Conn_01x13
- removed J?: Conn_01x08, symbol Connector_Generic:Conn_01x08
- removed R? (x13): 220K, symbol Device:R
- removed R?: 330, symbol Device:R
- removed R? (x6): 47K, symbol Device:R
- removed SW? (x13): SW_Push, symbol Switch:SW_Push
- removed U?: PAM8403, symbol pam8403:PAM8403
- added C? (x2): 470nF, Capacitor_SMD:C_0603_1608Metric_Pad1.05x0.95mm_HandSolder, symbol Device:C
- added C? (x3): 1uF, Capacitor_SMD:C_0603_1608Metric_Pad1.05x0.95mm_HandSolder, symbol Device:C
- added C?: 100nF, Capacitor_SMD:C_0603_1608Metric_Pad1.05x0.95mm_HandSolder, symbol Device:C
- added C?: 470uF, Capacitor_SMD:C_0603_1608Metric_Pad1.05x0.95mm_HandSolder, symbol Device:C
- added LS? (x2): Speaker, symbol Device:Speaker
- added R? (x2): 62K, Resistor_SMD:R_0603_1608Metric_Pad1.05x0.95mm_HandSolder, symbol Device:R
- added R? (x6): 47K, Resistor_SMD:R_0603_1608Metric_Pad1.05x0.95mm_HandSolder, symbol Device:R
- added RV?: 10K, wolf_lib:Potentiometer_Dual_5pin, symbol wolf_lib:R_POT_Dual_5pin
- added SW? (x13): SW_Push, wolf_lib:contact_button, symbol Switch:SW_Push
- added U?: PAM8403, Package_SO:SOP-16_4.4x10.4mm_P1.27mm, symbol wolf_lib:PAM8403
- added XS1: SD_Holder_TFP09-2-12B, wolf_lib:TFP09-2-12B, symbol wolf_lib:SD_Holder_TFP09-2-12B
- C1, C10, C11, C12, C2, C3, C4, C5, C6, C7, C8, C9: renamed from C?; footprint (none) -> Capacitor_SMD:C_0603_1608Metric_Pad1.05x0.95mm_HandSolder
- D1: renamed from D?; footprint (none) -> LED_SMD:LED_0603_1608Metric_Pad1.05x0.95mm_HandSolder
- J1: renamed from J?; footprint (none) -> Connector_USB:USB_Micro-B_Molex-105017-0001
- J3: renamed from J?; footprint (none) -> wolf_lib:OLED_SSD1325_2.7in
- J5, J6: renamed from J?; footprint (none) -> Connector_PinHeader_2.54mm:PinHeader_1x03_P2.54mm_Vertical
- R1, R2, R3, R4, R5, R6: renamed from R?; footprint (none) -> Resistor_SMD:R_0603_1608Metric_Pad1.05x0.95mm_HandSolder
- SW1, SW2: renamed from SW?; footprint (none) -> wolf_lib:contact_button
- U1: renamed from U?; footprint (none) -> Package_TO_SOT_SMD:SOT-223
- Y1, Y2: renamed from Y?; footprint (none) -> Crystal:Crystal_HC52-6mm_Vertical
- gave numbers to parts that had none: 1
Connections:
- net labels added: BTN_A, BTN_B, BTN_C, BTN_DD, BTN_DL, BTN_DR, BTN_DU, BTN_LT, BTN_Menu, BTN_RT, BTN_X, BTN_Y, BTN_Z, USB_D+, USB_D-
- net labels removed: BTN_0, BTN_1, BTN_10, BTN_11, BTN_12, BTN_2, BTN_3, BTN_4, BTN_5, BTN_6, BTN_7, BTN_8, BTN_9, USB_DM, USB_DP
- wire segments 255 -> 148
- no-connect marks 6 -> 7
Other:
- note added: "*Internal pull-up"
- note added: "AUDIO"
- note added: "BUTTONS"
- note removed: "KEYS"
- moved on the sheet: J3, J5, J6
